File: timer-display.kicad_pcb (KiCad board)
At the start: 2 copper layers, 107 x 92 mm, 62 parts, among them Q1 MBT3904DW1, Q10 IRLML6346, Q11 MBT3904DW1, Q12 IRLML6346, Q13 MBT3904DW1, Q14 IRLML6346, Q2 IRLML6346, Q3 MBT3904DW1, Q4 IRLML6346, Q5 MBT3904DW1, Q6 IRLML6346, Q7 MBT3904DW1, Q8 IRLML6346, Q9 MBT3904DW1, U1 SN74LS08, U2 SN74HC595DT, U3 SN74LS08

Commit message: production ready
Parts:
- added C4: 100n, Capacitor_SMD:C_0603_1608Metric, B.Cu at (244.5, 100.5)
- added C5: 100n, Capacitor_SMD:C_0603_1608Metric, B.Cu at (218.9, 109.0)
- added C6: 100n, Capacitor_SMD:C_0603_1608Metric, B.Cu at (247.2, 138.1)
- added D22: LTST-C171KRKT, LED_SMD:LED_0805_2012Metric, F.Cu at (222.5, 83.0)
- added D23: LTST-C171KRKT, LED_SMD:LED_0805_2012Metric, F.Cu at (222.5, 95.0)
- added D24: LTST-C171KRKT, LED_SMD:LED_0805_2012Metric, F.Cu at (222.5, 107.0)
- added D25: LTST-C171KRKT, LED_SMD:LED_0805_2012Metric, F.Cu at (230.5, 115.0)
- added D26: LTST-C171KRKT, LED_SMD:LED_0805_2012Metric, F.Cu at (242.5, 115.0)
- added D27: LTST-C171KRKT, LED_SMD:LED_0805_2012Metric, F.Cu at (254.5, 115.0)
- added D28: LTST-C171KRKT, LED_SMD:LED_0805_2012Metric, F.Cu at (254.5, 75.0)
- added D29: LTST-C171KRKT, LED_SMD:LED_0805_2012Metric, F.Cu at (242.5, 75.0)
- added D30: LTST-C171KRKT, LED_SMD:LED_0805_2012Metric, F.Cu at (230.5, 75.0)
- added D31: LTST-C171KRKT, LED_SMD:LED_0805_2012Metric, F.Cu at (262.5, 107.0)
- added D32: LTST-C171KRKT, LED_SMD:LED_0805_2012Metric, F.Cu at (262.5, 95.0)
- added D33: LTST-C171KRKT, LED_SMD:LED_0805_2012Metric, F.Cu at (262.5, 83.0)
- added D34: LTST-C171KRKT, LED_SMD:LED_0805_2012Metric, F.Cu at (230.5, 155.0)
- added D35: LTST-C171KRKT, LED_SMD:LED_0805_2012Metric, F.Cu at (242.5, 155.0)
- added D36: LTST-C171KRKT, LED_SMD:LED_0805_2012Metric, F.Cu at (254.5, 155.0)
- added D37: LTST-C171KRKT, LED_SMD:LED_0805_2012Metric, F.Cu at (262.5, 147.0)
- added D38: LTST-C171KRKT, LED_SMD:LED_0805_2012Metric, F.Cu at (262.5, 135.0)
- added D39: LTST-C171KRKT, LED_SMD:LED_0805_2012Metric, F.Cu at (262.5, 123.0)
- added D40: LTST-C171KRKT, LED_SMD:LED_0805_2012Metric, F.Cu at (222.5, 123.0)
- added D41: LTST-C171KRKT, LED_SMD:LED_0805_2012Metric, F.Cu at (222.5, 135.0)
- added D42: LTST-C171KRKT, LED_SMD:LED_0805_2012Metric, F.Cu at (222.5, 147.0)
- added H1: MountingHole, MountingHole:MountingHole_3.2mm_M3, F.Cu at (165.0, 72.5)
- added H2: MountingHole, MountingHole:MountingHole_3.2mm_M3, F.Cu at (265.0, 72.5)
- added H3: MountingHole, MountingHole:MountingHole_3.2mm_M3, F.Cu at (265.0, 157.5)
- added H4: MountingHole, MountingHole:MountingHole_3.2mm_M3, F.Cu at (165.0, 157.5)
- added J1: PWR, Connector_PinSocket_2.54mm:PinSocket_1x03_P2.54mm_Vertical, B.Cu at (198.0, 146.2)
- added J2: IN, Connector_PinSocket_1.27mm:PinSocket_1x06_P1.27mm_Vertical, B.Cu at (212.5, 152.3)
- added J3: OUT, Connector_PinSocket_1.27mm:PinSocket_1x06_P1.27mm_Vertical, B.Cu at (217.5, 152.3)
- added Q15: MBT3904DW1, Package_TO_SOT_SMD:SOT-363_SC-70-6, B.Cu at (221.1, 101.2)
- added Q16: T2N7002AK,LM, Package_TO_SOT_SMD:SOT-23, B.Cu at (224.3, 100.9)
- added Q17: MBT3904DW1, Package_TO_SOT_SMD:SOT-363_SC-70-6, B.Cu at (248.9, 116.4)
- added Q18: T2N7002AK,LM, Package_TO_SOT_SMD:SOT-23, B.Cu at (248.6, 113.2)
- added Q19: MBT3904DW1, Package_TO_SOT_SMD:SOT-363_SC-70-6, B.Cu at (236.5, 73.5)
- added Q20: T2N7002AK,LM, Package_TO_SOT_SMD:SOT-23, B.Cu at (236.8, 76.7)
- added Q21: MBT3904DW1, Package_TO_SOT_SMD:SOT-363_SC-70-6, B.Cu at (264.0, 88.7)
- added Q22: T2N7002AK,LM, Package_TO_SOT_SMD:SOT-23, B.Cu at (260.8, 89.0)
- added Q23: MBT3904DW1, Package_TO_SOT_SMD:SOT-363_SC-70-6, B.Cu at (249.0, 156.4)
- added Q24: T2N7002AK,LM, Package_TO_SOT_SMD:SOT-23, B.Cu at (248.7, 153.2)
- added Q25: MBT3904DW1, Package_TO_SOT_SMD:SOT-363_SC-70-6, B.Cu at (264.0, 128.6)
- added Q26: T2N7002AK,LM, Package_TO_SOT_SMD:SOT-23, B.Cu at (260.7, 128.9)
- added Q27: MBT3904DW1, Package_TO_SOT_SMD:SOT-363_SC-70-6, B.Cu at (221.0, 141.2)
- added Q28: T2N7002AK,LM, Package_TO_SOT_SMD:SOT-23, B.Cu at (224.2, 141.0)
- added R22: 10k, Resistor_SMD:R_0603_1608Metric, B.Cu at (221.0, 98.7)
- added R23: 1k, Resistor_SMD:R_0603_1608Metric, B.Cu at (224.2, 98.1)
- added R24: 36, Resistor_SMD:R_0603_1608Metric, B.Cu at (221.5, 103.7)
- added R25: 10k, Resistor_SMD:R_0603_1608Metric, B.Cu at (246.4, 116.5)
- added R26: 1k, Resistor_SMD:R_0603_1608Metric, B.Cu at (245.8, 113.3)
- added R27: 36, Resistor_SMD:R_0603_1608Metric, B.Cu at (251.4, 116.0)
- added R28: 10k, Resistor_SMD:R_0603_1608Metric, B.Cu at (239.0, 73.3)
- added R29: 1k, Resistor_SMD:R_0603_1608Metric, B.Cu at (239.6, 76.6)
- added R30: 36, Resistor_SMD:R_0603_1608Metric, B.Cu at (234.0, 73.9)
- added R31: 10k, Resistor_SMD:R_0603_1608Metric, B.Cu at (264.1, 91.2)
- added R32: 1k, Resistor_SMD:R_0603_1608Metric, B.Cu at (261.0, 91.8)
- added R33: 36, Resistor_SMD:R_0603_1608Metric, B.Cu at (263.7, 86.2)
- added R34: 10k, Resistor_SMD:R_0603_1608Metric, B.Cu at (246.5, 156.6)
- added R35: 1k, Resistor_SMD:R_0603_1608Metric, B.Cu at (245.9, 153.3)
- added R36: 36, Resistor_SMD:R_0603_1608Metric, B.Cu at (251.5, 156.0)
- added R37: 10k, Resistor_SMD:R_0603_1608Metric, B.Cu at (264.0, 131.1)
- added R38: 1k, Resistor_SMD:R_0603_1608Metric, B.Cu at (260.8, 131.7)
- added R39: 36, Resistor_SMD:R_0603_1608Metric, B.Cu at (263.7, 126.1)
- added R40: 10k, Resistor_SMD:R_0603_1608Metric, B.Cu at (220.9, 138.8)
- added R41: 1k, Resistor_SMD:R_0603_1608Metric, B.Cu at (224.1, 138.2)
- added R42: 36, Resistor_SMD:R_0603_1608Metric, B.Cu at (221.3, 143.8)
- added R43: 100k, Resistor_SMD:R_0603_1608Metric, B.Cu at (226.8, 99.0)
- added R44: 100k, Resistor_SMD:R_0603_1608Metric, B.Cu at (246.7, 110.7)
- added R45: 100k, Resistor_SMD:R_0603_1608Metric, B.Cu at (238.8, 79.2)
- added R46: 100k, Resistor_SMD:R_0603_1608Metric, B.Cu at (258.2, 91.0)
- added R47: 100k, Resistor_SMD:R_0603_1608Metric, B.Cu at (246.8, 150.7)
- added R48: 100k, Resistor_SMD:R_0603_1608Metric, B.Cu at (258.1, 130.8)
- added R49: 100k, Resistor_SMD:R_0603_1608Metric, B.Cu at (226.8, 139.1)
- added R50: 100k, Resistor_SMD:R_0603_1608Metric, B.Cu at (183.2, 79.3)
- added R51: 100k, Resistor_SMD:R_0603_1608Metric, B.Cu at (203.2, 90.9)
- added R52: 100k, Resistor_SMD:R_0603_1608Metric, B.Cu at (191.6, 110.8)
- added R53: 100k, Resistor_SMD:R_0603_1608Metric, B.Cu at (171.8, 99.0)
- added R54: 100k, Resistor_SMD:R_0603_1608Metric, B.Cu at (191.8, 150.8)
- added R55: 100k, Resistor_SMD:R_0603_1608Metric, B.Cu at (171.8, 138.9)
- added R56: 100k, Resistor_SMD:R_0603_1608Metric, B.Cu at (203.2, 130.9)
- added REF**: KiCad-Logo2_6mm_SilkScreen, Symbol:KiCad-Logo2_6mm_SilkScreen, F.Cu at (181.9, 84.2)
- added REF**: OSHW-Logo2_9.8x8mm_SilkScreen, Symbol:OSHW-Logo2_9.8x8mm_SilkScreen, F.Cu at (251.0, 85.2)
- added REF**: KiCad-Logo2_6mm_SilkScreen, Symbol:KiCad-Logo2_6mm_SilkScreen, B.Cu at (248.2, 84.2)
- added REF**: OSHW-Logo2_9.8x8mm_SilkScreen, Symbol:OSHW-Logo2_9.8x8mm_SilkScreen, B.Cu at (178.9, 85.2)
- added U4: SN74LS08, Package_SO:SOIC-14_3.9x8.7mm_P1.27mm, B.Cu at (242.5, 95.0)
- added U5: SN74HC595DT, Package_SO:SOIC-16_3.9x9.9mm_P1.27mm, B.Cu at (222.0, 115.0)
- added U6: SN74LS08, Package_SO:SOIC-14_3.9x8.7mm_P1.27mm, B.Cu at (242.5, 135.0)
- Q10, Q12, Q14, Q2, Q4, Q6, Q8: value IRLML6346 -> T2N7002AK,LM
- R11, R14, R17, R2, R20, R5, R8: value 10 -> 1k
- moved U2 1.00 mm to (208.0, 115.0)
- moved C3 0.75 mm to (211.0, 121.0)
Connections:
- net /Digit-MinuteTen/A renamed /Digit-Ten/A
- net /Digit-MinuteTen/Araw renamed /Digit-Ten/Araw
- net /Digit-MinuteTen/B renamed /Digit-Ten/B
- net /Digit-MinuteTen/Braw renamed /Digit-Ten/Braw
- net /Digit-MinuteTen/C renamed /Digit-Ten/C
- net /Digit-MinuteTen/Craw renamed /Digit-Ten/Craw
- net /Digit-MinuteTen/D renamed /Digit-Ten/D
- net /Digit-MinuteTen/Draw renamed /Digit-Ten/Draw
- net /Digit-MinuteTen/E renamed /Digit-Ten/E
- net /Digit-MinuteTen/Eraw renamed /Digit-Ten/Eraw
- net /Digit-MinuteTen/F renamed /Digit-Ten/F
- net /Digit-MinuteTen/Fraw renamed /Digit-Ten/Fraw
- net /Digit-MinuteTen/G renamed /Digit-Ten/G
- net /Digit-MinuteTen/Graw renamed /Digit-Ten/Graw
- U2 pad 9: /Digit-MinuteTen/SERout -> /Digit-One/SERin
Routing:
- net +12V: track 295.3 -> 607.3 mm, vias 7 -> 18
- net PWM: track 71.9 -> 285.0 mm, vias 0 -> 2
- net +5V: track 84.3 -> 197.0 mm, vias 0 -> 4
- net SERclr: track 0.00 -> 61.9 mm
- net SERclk: track 0.00 -> 58.5 mm, vias 0 -> 2
- net GND: track 34.4 -> 92.5 mm, vias 13 -> 26
- net REGclr: track 0.00 -> 56.7 mm, vias 0 -> 2
- net OE: track 0.00 -> 55.4 mm, vias 0 -> 2
- net /Digit-One/Araw: track 0.00 -> 46.3 mm
- net /Digit-One/Draw: track 0.00 -> 43.7 mm, vias 0 -> 4
- net /Digit-One/Braw: track 0.00 -> 40.5 mm
- net /Digit-One/Craw: track 0.00 -> 38.5 mm, vias 0 -> 4
- net /Digit-One/Eraw: track 0.00 -> 38.2 mm, vias 0 -> 4
- net Serial: track 0.00 -> 37.7 mm
- net SerialOut: track 0.00 -> 35.1 mm
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Other:
- outline, holes or cut-outs redrawn
- board text added: "*"
- board text added: "12V 5V GND"
- board text added: "Input / Output: 1 Serial In/Out 2 OutEnable 3 RegClock 4 SerialClock 5 SerialClear 6 PWM"
- board text added: "Input/Output: 1 SerialIn/Out 2 OutEnable 3 RegClock 4 SerialClock 5 SerialClear 6 PWM"
- board text added: "SendOffTimer v1.1 10/22 by scottec"

Commit message: 7.0.1 -> 7.0.10
Other:
- board text added: "locked"
