File: timer-display.kicad_sch (KiCad schematic)
At the start: 0 parts

Commit message: production ready
Parts:
- added H1, H2, H3, H4: MountingHole, MountingHole:MountingHole_3.2mm_M3, symbol Mechanical:MountingHole
- added J1: PWR, Connector_PinSocket_2.54mm:PinSocket_1x03_P2.54mm_Vertical, symbol Connector_Generic:Conn_01x03
- added J2: IN, Connector_PinSocket_1.27mm:PinSocket_1x06_P1.27mm_Vertical, symbol Connector_Generic:Conn_01x06
- added J3: OUT, Connector_PinSocket_1.27mm:PinSocket_1x06_P1.27mm_Vertical, symbol Connector_Generic:Conn_01x06
Connections:
- net OE: now also J2.2 (Pin_2), J3.2 (Pin_2)
- net PWM: now also J2.6 (Pin_6), J3.6 (Pin_6)
- net REGclr: now also J2.3 (Pin_3), J3.3 (Pin_3)
- net SERclk: now also J2.4 (Pin_4), J3.4 (Pin_4)
- net SERclr: now also J2.5 (Pin_5), J3.5 (Pin_5)
- net Serial: now also J2.1 (Pin_1)
- new net +12V: J1.1 (Pin_1)
- new net +5V: J1.2 (Pin_2)
- new net GND: J1.3 (Pin_3)
- new net SerialOut: J3.1 (Pin_1)
Other:
- sheet Digit-MinuteTen renamed Digit-Ten
- added sheet Digit-One (timer-display-digit.kicad_sch)
